File: system_development/Cellular/v0.2/Custom PCB's/Power PCB/Power PCB.kicad_pcb (KiCad board)
At the start: 2 copper layers, 30.5 x 53.3 mm, 14 parts, among them J1 Barrel_Jack, SW1 SW_DIP_x01, U1 LF15_TO252, U2 INA219A

Commit message: PCB updates
Updated Power PCB so that INA219 chip is connected to ground and has a stable I2C address. Updated datalogging board with a bigger 3.3V regulator since the previous tiny one was not working in the board.
Connections:
- U2 pad 1: unconnected-(U2-A1-Pad1) -> GND
- U2 pad 2: unconnected-(U2-A0-Pad2) -> GND
